Commit message: phase 1 including lidar and bot and obstacle detection completed

File: install/mobile_robot/share/mobile_robot/model/robot.xacro (robot description, xacro)
@@ -2,5 +2,5 @@
 <robot name="differential_drive_robot" xmlns:xacro="http://www.ros.org/wiki/xacro">
 <xacro:property name="pi_const" value="3.14159265358979323846"/>
-<xacro:propery name="a" value="1.0"/>
+<xacro:property name="a" value="1.0"/>
 <xacro:property name="b" value="0.3"/>
 <xacro:property name="c" value="0.6"/>
@@ -18,29 +18,29 @@
 <xacro:property name="m3" value="${d3*(4.0/3.0)*pi_const*r*r*r}"/>
 <xacro:property name="Ix_body" value="${(1.0/12.0)*m1*(b*b+c*c)}"/>
-<xacro:property name="Iy_body" value="${(1.0/12.0)*m1*(a*a+b*b)}"/>
-<xacro:property name="Iz_body" value="${(1.0/12.0)*m1*(a*a+c*c)}"/>
+<xacro:property name="Iy_body" value="${(1.0/12.0)*m1*(a*a+c*c)}"/>
+<xacro:property name="Iz_body" value="${(1.0/12.0)*m1*(a*a+b*b)}"/>
 <xacro:property name="Iz_wheel" value="${(1.0/2.0)*m2*r*r}"/>
 <xacro:property name="I_wheel" value="${(1.0/12.0)*m2*(3.0*r*r+d*d)}"/>
 <xacro:property name="I_caster" value="${(2.0/5.0)*m3*r*r}"/>
 <xacro:macro name="inertia_body">
-        <intertial>
+        <inertial>
         <origin rpy="0 0 0" xyz="0 0 ${s1}" />
         <mass value="${m1}" />
-        <inertia ixx="${Ix_body}" ixy="0.0" ixz="0.0" iyy="${Iy_body}" iyz="0.0" izz="${Iy_body}" iyz="0" izz="${Iz_body}" />
-        </intertial>
+        <inertia ixx="${Ix_body}" ixy="0.0" ixz="0.0" iyy="${Iy_body}" iyz="0.0" izz="${Iz_body}" />
+        </inertial>
 </xacro:macro>
 <xacro:macro name="inertia_wheel">
-        <intertial>
+        <inertial>
         <origin rpy="1.570795 0 0" xyz="0 0 0" />
         <mass value="${m2}" />
         <inertia ixx="${I_wheel}" ixy="0.0" ixz="0.0" iyy="${I_wheel}" iyz="0.0" izz="${Iz_wheel}" />
-        </intertial>
+        </inertial>
 </xacro:macro>
 <xacro:macro name="inertia_caster">
-        <intertial>
+        <inertial>
         <origin rpy="0 0 0" xyz="0 0 0" />
         <mass value="${m3}" />
         <inertia ixx="${I_caster}" ixy="0.0" ixz="0.0" iyy="${I_caster}" iyz="0.0" izz="${I_caster}" />
-        </intertial>
+        </inertial>
 </xacro:macro>
 <xacro:include filename="$(find mobile_robot)/model/robot.gazebo" />
@@ -67,5 +67,5 @@
 <joint name="wheel1_joint" type="continuous">
     <parent link="body_link"/>
-    <child link="wheell1_link"/>
+    <child link="wheel1_link"/>
     <origin rpy="0 0 0" xyz="${-s2} ${-s4} ${r}"/>
     <axis xyz="0 1 0"/>
@@ -134,5 +134,5 @@
     <parent link="body_link"/>
     <child link="lidar_link"/>
-    <origin rpy="0 0 0" xyz="0.0 0 ${b+r}"/>
+    <origin rpy="0 0 0" xyz="0.0 0 0.62"/>
     <axis xyz="0 1 0" rpy="0 0 0"/>
 </joint>
@@ -151,5 +151,5 @@
     </collision>
     <inertial>
-        <mass value="1e-6">
+        <mass value="1e-6" />
         <origin xyz="0 0 0" rpy="0 0 0" />
         <inertia ixx="1e-6" ixy="0" ixz="0"

Commit message: gazebo rviz slam_toolbox working properly

File: install/mobile_robot/share/mobile_robot/model/robot.xacro (robot description, xacro)
@@ -111,5 +111,5 @@
     <xacro:inertia_wheel/>
 </link>
-<joint name="caster_joint" type="continuous">
+<joint name="caster_joint" type="fixed">
     <parent link="body_link"/>
     <child link="caster_link"/>

Commit message: configuring nav2 brain of the bot

File: install/mobile_robot/share/mobile_robot/model/robot.xacro (robot description, xacro)
@@ -1,160 +1 @@
-<?xml version="1.0"?>
-<robot name="differential_drive_robot" xmlns:xacro="http://www.ros.org/wiki/xacro">
-<xacro:property name="pi_const" value="3.14159265358979323846"/>
-<xacro:property name="a" value="1.0"/>
-<xacro:property name="b" value="0.3"/>
-<xacro:property name="c" value="0.6"/>
-<xacro:property name="r" value="0.15"/>
-<xacro:property name="d" value="0.1"/>
-<xacro:property name="s1" value="${b/2+r}"/>
-<xacro:property name="s2" value="${2*r}"/>
-<xacro:property name="s3" value="${2*r}"/>
-<xacro:property name="s4" value="${c/2+d/2}"/>
-<xacro:property name="d1" value="2710.0"/>
-<xacro:property name="d2" value="2710.0"/>
-<xacro:property name="d3" value="2710.0"/>
-<xacro:property name="m1" value="${d1*a*b*c}"/>
-<xacro:property name="m2" value="${d2*pi_const*r*r*d}"/>
-<xacro:property name="m3" value="${d3*(4.0/3.0)*pi_const*r*r*r}"/>
-<xacro:property name="Ix_body" value="${(1.0/12.0)*m1*(b*b+c*c)}"/>
-<xacro:property name="Iy_body" value="${(1.0/12.0)*m1*(a*a+c*c)}"/>
-<xacro:property name="Iz_body" value="${(1.0/12.0)*m1*(a*a+b*b)}"/>
-<xacro:property name="Iz_wheel" value="${(1.0/2.0)*m2*r*r}"/>
-<xacro:property name="I_wheel" value="${(1.0/12.0)*m2*(3.0*r*r+d*d)}"/>
-<xacro:property name="I_caster" value="${(2.0/5.0)*m3*r*r}"/>
-<xacro:macro name="inertia_body">
-        <inertial>
-        <origin rpy="0 0 0" xyz="0 0 ${s1}" />
-        <mass value="${m1}" />
-        <inertia ixx="${Ix_body}" ixy="0.0" ixz="0.0" iyy="${Iy_body}" iyz="0.0" izz="${Iz_body}" />
-        </inertial>
-</xacro:macro>
-<xacro:macro name="inertia_wheel">
-        <inertial>
-        <origin rpy="1.570795 0 0" xyz="0 0 0" />
-        <mass value="${m2}" />
-        <inertia ixx="${I_wheel}" ixy="0.0" ixz="0.0" iyy="${I_wheel}" iyz="0.0" izz="${Iz_wheel}" />
-        </inertial>
-</xacro:macro>
-<xacro:macro name="inertia_caster">
-        <inertial>
-        <origin rpy="0 0 0" xyz="0 0 0" />
-        <mass value="${m3}" />
-        <inertia ixx="${I_caster}" ixy="0.0" ixz="0.0" iyy="${I_caster}" iyz="0.0" izz="${I_caster}" />
-        </inertial>
-</xacro:macro>
-<xacro:include filename="$(find mobile_robot)/model/robot.gazebo" />
-<link name="base_footprint"></link>
-<joint name="body_link_joint" type="fixed">
-    <parent link="base_footprint"/>
-    <child link="body_link"/>
-</joint>
-<link name="body_link">
-    <visual>
-        <geometry>
-            <box size="${a} ${b} ${c}" />
-        </geometry>
-    <origin rpy="0.0 0.0 0.0" xyz="0.0 0.0 ${s1}"/>
-    </visual>
-    <collision>
-        <geometry>
-            <box size="${a} ${b} ${c}" />
-        </geometry>
-        <origin rpy="0 0 0" xyz="0 0 ${s1}" />
-    </collision>
-    <xacro:inertia_body/>
-</link>
-<joint name="wheel1_joint" type="continuous">
-    <parent link="body_link"/>
-    <child link="wheel1_link"/>
-    <origin rpy="0 0 0" xyz="${-s2} ${-s4} ${r}"/>
-    <axis xyz="0 1 0"/>
-    <limit effort="50000" velocity="10.0"/>
-    <dynamics damping="1.0" friction="1.0"/>
-</joint>
-<link name="wheel1_link">
-    <visual>
-        <geometry>
-            <cylinder radius="${r}" length="${d}"/>
-        </geometry>
-        <origin rpy="1.570795 0 0" xyz="0 0 0"/>
-    </visual>
-    <collision>
-        <geometry>
-            <cylinder radius="${r}" length="${d}"/>
-        </geometry>
-        <origin rpy="1.570795 0 0" xyz="0 0 0"/>
-    </collision>
-    <xacro:inertia_wheel/>
-</link>
-<joint name="wheel2_joint" type="continuous">
-    <parent link="body_link"/>
-    <child link="wheel2_link"/>
-    <origin rpy="0 0 0" xyz="${-s2} ${s4} ${r}"/>
-    <axis xyz="0 1 0"/>
-    <limit effort="50000" velocity="10.0"/>
-    <dynamics damping="1.0" friction="1.0"/>
-</joint>
-<link name="wheel2_link">
-    <visual>
-        <geometry>
-            <cylinder radius="${r}" length="${d}"/>
-        </geometry>
-        <origin rpy="1.570795 0 0" xyz="0 0 0"/>
-    </visual>
-    <collision>
-        <geometry>
-            <cylinder radius="${r}" length="${d}"/>
-        </geometry>
-        <origin rpy="1.570795 0 0" xyz="0 0 0"/>
-    </collision>
-    <xacro:inertia_wheel/>
-</link>
-<joint name="caster_joint" type="fixed">
-    <parent link="body_link"/>
-    <child link="caster_link"/>
-    <origin rpy="0 0 0" xyz="${s3} 0 ${r}"/>
-</joint>
-<link name="caster_link">
-    <visual>
-        <geometry>
-            <sphere radius="${r}"/>
-        </geometry>
-        <origin rpy="0 0 0" xyz="0 0 0"/>
-    </visual>
-    <collision>
-        <geometry>
-            <sphere radius="${r}"/>
-        </geometry>
-        <origin rpy="0 0 0" xyz="0 0 0"/>
-    </collision>
-    <xacro:inertia_caster/>
-</link>
-<joint name="lidar_joint" type="fixed">
-    <parent link="body_link"/>
-    <child link="lidar_link"/>
-    <origin rpy="0 0 0" xyz="0.0 0 0.62"/>
-    <axis xyz="0 1 0" rpy="0 0 0"/>
-</joint>
-<link name="lidar_link">
-    <visual>
-        <geometry>
-            <cylinder radius="0.1" length="0.1"/>
-        </geometry>
-        <origin rpy="0 0 0.05" xyz="0 0 0"/>
-    </visual>
-    <collision>
-        <geometry>
-            <cylinder radius="0.1" length="0.1"/>
-        </geometry>
-        <origin rpy="0 0 0.05" xyz="0 0 0"/>
-    </collision>
-    <inertial>
-        <mass value="1e-6" />
-        <origin xyz="0 0 0" rpy="0 0 0" />
-        <inertia ixx="1e-6" ixy="0" ixz="0"
-                            iyy="1e-6" iyz="0" izz="1e-6"
-        />
-        </inertial>
-</link>
-</robot>
+/home/pouryajafari/ws_mobile/build/mobile_robot/model/robot.xacro

File: src/mobile_robot/model/robot.xacro (robot description, xacro)
@@ -7,11 +7,11 @@
 <xacro:property name="r" value="0.15"/>
 <xacro:property name="d" value="0.1"/>
-<xacro:property name="s1" value="${b/2+r}"/>
+<xacro:property name="s1" value="${b/2+r+0.05}"/>
 <xacro:property name="s2" value="${2*r}"/>
 <xacro:property name="s3" value="${2*r}"/>
 <xacro:property name="s4" value="${c/2+d/2}"/>
-<xacro:property name="d1" value="2710.0"/>
-<xacro:property name="d2" value="2710.0"/>
-<xacro:property name="d3" value="2710.0"/>
+<xacro:property name="d1" value="500.0"/>
+<xacro:property name="d2" value="1000.0"/>
+<xacro:property name="d3" value="1000.0"/>
 <xacro:property name="m1" value="${d1*a*b*c}"/>
 <xacro:property name="m2" value="${d2*pi_const*r*r*d}"/>
@@ -69,5 +69,5 @@
     <child link="wheel1_link"/>
     <origin rpy="0 0 0" xyz="${-s2} ${-s4} ${r}"/>
-    <axis xyz="0 1 0"/>
+    <axis xyz="0 -1 0"/>
     <limit effort="50000" velocity="10.0"/>
     <dynamics damping="1.0" friction="1.0"/>
@@ -92,5 +92,5 @@
     <child link="wheel2_link"/>
     <origin rpy="0 0 0" xyz="${-s2} ${s4} ${r}"/>
-    <axis xyz="0 1 0"/>
+    <axis xyz="0 -1 0"/>
     <limit effort="50000" velocity="10.0"/>
     <dynamics damping="1.0" friction="1.0"/>
@@ -151,10 +151,13 @@
     </collision>
     <inertial>
-        <mass value="1e-6" />
+        <mass value="0.1" />
         <origin xyz="0 0 0" rpy="0 0 0" />
-        <inertia ixx="1e-6" ixy="0" ixz="0"
-                            iyy="1e-6" iyz="0" izz="1e-6"
-        />
-        </inertial>
+        <inertia ixx="0.001" ixy="0" ixz="0"
+                 iyy="0.001" iyz="0" izz="0.001" />
+    </inertial>
 </link>
+<gazebo reference="caster_link">
+    <mu1>0.0</mu1>
+    <mu2>0.0</mu2>
+</gazebo>
 </robot>
