Commit message: fixing the shape of the bot and its mass and inertia and adding to the lidar range

File: src/mobile_robot/model/robot.xacro (robot description, xacro)
@@ -7,11 +7,11 @@
 <xacro:property name="r" value="0.15"/>
 <xacro:property name="d" value="0.1"/>
-<xacro:property name="s1" value="${b/2+r+0.05}"/>
+<xacro:property name="s1" value="${b/2+r}"/>
 <xacro:property name="s2" value="${2*r}"/>
 <xacro:property name="s3" value="${2*r}"/>
-<xacro:property name="s4" value="${c/2+d/2}"/>
-<xacro:property name="d1" value="500.0"/>
-<xacro:property name="d2" value="1000.0"/>
-<xacro:property name="d3" value="1000.0"/>
+<xacro:property name="s4" value="${b/2 + d/2 + 0.02}"/>
+<xacro:property name="d1" value="50.0"/>
+<xacro:property name="d2" value="50.0"/>
+<xacro:property name="d3" value="50.0"/>
 <xacro:property name="m1" value="${d1*a*b*c}"/>
 <xacro:property name="m2" value="${d2*pi_const*r*r*d}"/>
@@ -69,6 +69,6 @@
     <child link="wheel1_link"/>
     <origin rpy="0 0 0" xyz="${-s2} ${-s4} ${r}"/>
-    <axis xyz="0 -1 0"/>
-    <limit effort="50000" velocity="10.0"/>
+    <axis xyz="0 1 0"/>
+    <limit effort="100" velocity="10.0"/>
     <dynamics damping="1.0" friction="1.0"/>
 </joint>
@@ -92,6 +92,6 @@
     <child link="wheel2_link"/>
     <origin rpy="0 0 0" xyz="${-s2} ${s4} ${r}"/>
-    <axis xyz="0 -1 0"/>
-    <limit effort="50000" velocity="10.0"/>
+    <axis xyz="0 1 0"/>
+    <limit effort="100" velocity="10.0"/>
     <dynamics damping="1.0" friction="1.0"/>
 </joint>
@@ -142,5 +142,5 @@
             <cylinder radius="0.1" length="0.1"/>
         </geometry>
-        <origin rpy="0 0 0.05" xyz="0 0 0"/>
+        <origin rpy="0 0 0" xyz="0 0 0"/>
     </visual>
     <collision>
@@ -148,5 +148,5 @@
             <cylinder radius="0.1" length="0.1"/>
         </geometry>
-        <origin rpy="0 0 0.05" xyz="0 0 0"/>
+        <origin rpy="0 0 0" xyz="0 0 0"/>
     </collision>
     <inertial>
